File: hardware/pHAT/pHAT.sch (KiCad schematic (older format))
At the start: 20 parts, among them J0 Conn_01x04, J1 Conn_01x02, P1 Conn_02x20_Odd_Even, Q1 2N7002, U2 HIH6131-021, U3 P82B96

Commit message: Polishing the board
Other:
- note removed: "ID_SD and ID_SC PINS:\nThese pins are reserved for HAT ID EEPROM.\n\nAt boot time this I2C interface will be\ninterrogated to look for an EEPROM\nthat identifes the attached board and\nallows automagic setup of the GPIOs\n(and optionally, Linux drivers).\n\nDO NOT USE these pins for anything other\nthan attaching an I2C ID EEPROM. Leave\nunconnected if ID EEPROM not required."
Changed lines of the file:
@@
 Sheet 1 1
 Title "Beehive pHAT"
-Date "2019-03-12"
+Date "2019-03-20"
 Rev "v3.3"
 Comp "University of Glasgow"
-Comment1 ""
+Comment1 "ENG5220-RTEP"
 Comment2 ""
 Comment3 ""
@@
 	3100 1300 2900 1300
 Connection ~ 3100 1700
-Text Notes 650  7600 0    50   ~ 0
-ID_SD and ID_SC PINS:\nThese pins are reserved for HAT ID EEPROM.\n\nAt boot time this I2C interface will be\ninterrogated to look for an EEPROM\nthat identifes the attached board and\nallows automagic setup of the GPIOs\n(and optionally, Linux drivers).\n\nDO NOT USE these pins for anything other\nthan attaching an I2C ID EEPROM. Leave\nunconnected if ID EEPROM not required.
 $Comp
 L pHAT-rescue:Mounting_Hole-Mechanical MK1
